File: hardware/ledctl.kicad_pcb (KiCad board)
At the start: 2 copper layers, 64 x 38 mm, 36 parts, among them J1 DC_IN_12-24V, J2 LED_STRIP, J3 USB-C, J4 UART, Q1 AO3400A, SW1 RESET, SW2 BOOT/USER, U1 AP63203WU, U2 ESP32-C3-WROOM-02

Commit message: Add Bilginier branding and LCSC part numbers
- Bilginier circuit-brain logo (docs/logo/logo.py) as single source for
  SVG/banner, PCB silkscreen (add_branding.py) and engraved enclosure lid
- README banner with light/dark variants, schematic title block
- BOM.csv/BOM.md: verified LCSC numbers, JLCPCB BOM + CPL exports
- F1: flag that no 1812 PTC covers 3 A at 24 V (decision pending)

Co-Authored-By: Claude Opus 5.5 <noreply@anthropic.com>
Claude-Session: https://claude.ai/code/session_01N8odZzQsCCUC5sRgiuL7xi
Routing:
- net GND: vias 36 -> 28
Other:
- board text added: "BILGINIER rev A"
- board text added: "LED Controller"
- board text removed: "ESP32-C3 LED CTRL rev A"
