File: hardware/ledctl.kicad_sch (KiCad schematic)
At the start: 32 parts, among them J1 DC_IN_12-24V, J2 LED_STRIP, J3 USB-C, J4 UART, Q1 AO3400A, SW1 RESET, SW2 BOOT/USER, U1 AP63203WU, U2 ESP32-C3-WROOM-02

Commit message: Add Bilginier branding and LCSC part numbers
- Bilginier circuit-brain logo (docs/logo/logo.py) as single source for
  SVG/banner, PCB silkscreen (add_branding.py) and engraved enclosure lid
- README banner with light/dark variants, schematic title block
- BOM.csv/BOM.md: verified LCSC numbers, JLCPCB BOM + CPL exports
- F1: flag that no 1812 PTC covers 3 A at 24 V (decision pending)

Co-Authored-By: Claude Opus 5.5 <noreply@anthropic.com>
Claude-Session: https://claude.ai/code/session_01N8odZzQsCCUC5sRgiuL7xi
Other:
- company: (none) -> Bilginier
- title: ESP32-C3 LED Strip Controller -> LED Controller - ESP32-C3 LED Strip Controller
Changed lines of the file:
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@@
   (paper "A4")
   (title_block
-    (title "ESP32-C3 LED Strip Controller")
+    (title "LED Controller - ESP32-C3 LED Strip Controller")
     (rev "A")
+    (company "Bilginier")
     (comment 1 "12-24V LED serit, WiFi ac/kapa + PWM"))
   (symbol
@@
     (instances
       (project "ledctl"
-        (path "/946d1a7c-9394-4dcb-a7a9-b342a099c222"
+        (path "/32758bcc-8919-49fe-a557-bdc491a02cde"
           (reference "J1")
           (unit 1)))))
@@
     (instances
       (project "ledctl"
-        (path "/946d1a7c-9394-4dcb-a7a9-b342a099c222"
+        (path "/32758bcc-8919-49fe-a557-bdc491a02cde"
           (reference "F1")
           (unit 1)))))
@@
     (instances
       (project "ledctl"
-        (path "/946d1a7c-9394-4dcb-a7a9-b342a099c222"
+        (path "/32758bcc-8919-49fe-a557-bdc491a02cde"
           (reference "D3")
           (unit 1)))))
@@
     (instances
       (project "ledctl"
-        (path "/946d1a7c-9394-4dcb-a7a9-b342a099c222"
+        (path "/32758bcc-8919-49fe-a557-bdc491a02cde"
           (reference "J2")
           (unit 1)))))
@@
     (instances
       (project "ledctl"
-        (path "/946d1a7c-9394-4dcb-a7a9-b342a099c222"
+        (path "/32758bcc-8919-49fe-a557-bdc491a02cde"
           (reference "D1")
           (unit 1)))))
@@
     (instances
       (project "ledctl"
-        (path "/946d1a7c-9394-4dcb-a7a9-b342a099c222"
+        (path "/32758bcc-8919-49fe-a557-bdc491a02cde"
           (reference "D2")
           (unit 1)))))
@@
     (instances
       (project "ledctl"
-        (path "/946d1a7c-9394-4dcb-a7a9-b342a099c222"
+        (path "/32758bcc-8919-49fe-a557-bdc491a02cde"
           (reference "J3")
           (unit 1)))))
@@
     (instances
       (project "ledctl"
-        (path "/946d1a7c-9394-4dcb-a7a9-b342a099c222"
+        (path "/32758bcc-8919-49fe-a557-bdc491a02cde"
           (reference "R8")
           (unit 1)))))
@@
     (instances
       (project "ledctl"
-        (path "/946d1a7c-9394-4dcb-a7a9-b342a099c222"
+        (path "/32758bcc-8919-49fe-a557-bdc491a02cde"
           (reference "R9")
           (unit 1)))))
@@
     (instances
       (project "ledctl"
-        (path "/946d1a7c-9394-4dcb-a7a9-b342a099c222"
+        (path "/32758bcc-8919-49fe-a557-bdc491a02cde"
           (reference "U1")
           (unit 1)))))
@@
     (instances
       (project "ledctl"
-        (path "/946d1a7c-9394-4dcb-a7a9-b342a099c222"
+        (path "/32758bcc-8919-49fe-a557-bdc491a02cde"
           (reference "C1")
           (unit 1)))))
@@
     (instances
       (project "ledctl"
-        (path "/946d1a7c-9394-4dcb-a7a9-b342a099c222"
+        (path "/32758bcc-8919-49fe-a557-bdc491a02cde"
           (reference "C2")
           (unit 1)))))
@@
     (instances
       (project "ledctl"
-        (path "/946d1a7c-9394-4dcb-a7a9-b342a099c222"
+        (path "/32758bcc-8919-49fe-a557-bdc491a02cde"
           (reference "C3")
           (unit 1)))))
@@
     (instances
       (project "ledctl"
-        (path "/946d1a7c-9394-4dcb-a7a9-b342a099c222"
+        (path "/32758bcc-8919-49fe-a557-bdc491a02cde"
           (reference "L1")
           (unit 1)))))
@@
     (instances
       (project "ledctl"
-        (path "/946d1a7c-9394-4dcb-a7a9-b342a099c222"
+        (path "/32758bcc-8919-49fe-a557-bdc491a02cde"
           (reference "C4")
           (unit 1)))))
@@
     (instances
       (project "ledctl"
-        (path "/946d1a7c-9394-4dcb-a7a9-b342a099c222"
+        (path "/32758bcc-8919-49fe-a557-bdc491a02cde"
           (reference "C5")
           (unit 1)))))
@@
     (instances
       (project "ledctl"
-        (path "/946d1a7c-9394-4dcb-a7a9-b342a099c222"
+        (path "/32758bcc-8919-49fe-a557-bdc491a02cde"
           (reference "#FLG01")
           (unit 1)))))
@@
     (instances
       (project "ledctl"
-        (path "/946d1a7c-9394-4dcb-a7a9-b342a099c222"
+        (path "/32758bcc-8919-49fe-a557-bdc491a02cde"
           (reference "#FLG02")
           (unit 1)))))
@@
     (instances
       (project "ledctl"
-        (path "/946d1a7c-9394-4dcb-a7a9-b342a099c222"
+        (path "/32758bcc-8919-49fe-a557-bdc491a02cde"
           (reference "#FLG03")
           (unit 1)))))
@@
     (instances
       (project "ledctl"
-        (path "/946d1a7c-9394-4dcb-a7a9-b342a099c222"
+        (path "/32758bcc-8919-49fe-a557-bdc491a02cde"
           (reference "U2")
           (unit 1)))))
@@
     (instances
       (project "ledctl"
-        (path "/946d1a7c-9394-4dcb-a7a9-b342a099c222"
+        (path "/32758bcc-8919-49fe-a557-bdc491a02cde"
           (reference "C6")
           (unit 1)))))
@@
     (instances
       (project "ledctl"
-        (path "/946d1a7c-9394-4dcb-a7a9-b342a099c222"
+        (path "/32758bcc-8919-49fe-a557-bdc491a02cde"
           (reference "C7")
           (unit 1)))))
@@
     (instances
       (project "ledctl"
-        (path "/946d1a7c-9394-4dcb-a7a9-b342a099c222"
+        (path "/32758bcc-8919-49fe-a557-bdc491a02cde"
           (reference "R1")
           (unit 1)))))
@@
     (instances
       (project "ledctl"
-        (path "/946d1a7c-9394-4dcb-a7a9-b342a099c222"
+        (path "/32758bcc-8919-49fe-a557-bdc491a02cde"
           (reference "C8")
           (unit 1)))))
@@
     (instances
       (project "ledctl"
-        (path "/946d1a7c-9394-4dcb-a7a9-b342a099c222"
+        (path "/32758bcc-8919-49fe-a557-bdc491a02cde"
           (reference "SW1")
           (unit 1)))))
@@
     (instances
       (project "ledctl"
-        (path "/946d1a7c-9394-4dcb-a7a9-b342a099c222"
+        (path "/32758bcc-8919-49fe-a557-bdc491a02cde"
           (reference "R2")
           (unit 1)))))
@@
     (instances
       (project "ledctl"
-        (path "/946d1a7c-9394-4dcb-a7a9-b342a099c222"
+        (path "/32758bcc-8919-49fe-a557-bdc491a02cde"
           (reference "SW2")
           (unit 1)))))
@@
     (instances
       (project "ledctl"
-        (path "/946d1a7c-9394-4dcb-a7a9-b342a099c222"
+        (path "/32758bcc-8919-49fe-a557-bdc491a02cde"
           (reference "R3")
           (unit 1)))))
@@
     (instances
       (project "ledctl"
-        (path "/946d1a7c-9394-4dcb-a7a9-b342a099c222"
+        (path "/32758bcc-8919-49fe-a557-bdc491a02cde"
           (reference "R4")
           (unit 1)))))
@@
     (instances
       (project "ledctl"
-        (path "/946d1a7c-9394-4dcb-a7a9-b342a099c222"
+        (path "/32758bcc-8919-49fe-a557-bdc491a02cde"
           (reference "J4")
           (unit 1)))))
@@
     (instances
       (project "ledctl"
-        (path "/946d1a7c-9394-4dcb-a7a9-b342a099c222"
+        (path "/32758bcc-8919-49fe-a557-bdc491a02cde"
           (reference "R5")
           (unit 1)))))
@@
     (instances
       (project "ledctl"
-        (path "/946d1a7c-9394-4dcb-a7a9-b342a099c222"
+        (path "/32758bcc-8919-49fe-a557-bdc491a02cde"
           (reference "R6")
           (unit 1)))))
@@
     (instances
       (project "ledctl"
-        (path "/946d1a7c-9394-4dcb-a7a9-b342a099c222"
+        (path "/32758bcc-8919-49fe-a557-bdc491a02cde"
           (reference "Q1")
           (unit 1)))))
@@
     (instances
       (project "ledctl"
-        (path "/946d1a7c-9394-4dcb-a7a9-b342a099c222"
+        (path "/32758bcc-8919-49fe-a557-bdc491a02cde"
           (reference "R7")
           (unit 1)))))
@@
     (instances
       (project "ledctl"
-        (path "/946d1a7c-9394-4dcb-a7a9-b342a099c222"
+        (path "/32758bcc-8919-49fe-a557-bdc491a02cde"
           (reference "D4")
           (unit 1)))))
